File: kicad/phoenix-main-board/phoenix-main-board.kicad_sch (KiCad schematic)
At the start: 88 parts, among them U1 LM7705, U2 LT3092xDD, U3 TPS61222DCK, U4 Adafruit_Feather_nrf52840_Exp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, U5 TS5A3359, U6 TPS7A2033DQN, U7 OPA2380, U8 AD5242, U9 MCP3564

Commit message: PCB: Complete V1.0.1 Tsunami
Parts:
- added TP29: TestPoint_Small, TestPoint:TestPoint_Keystone_5000-5004_Miniature, symbol Connector:TestPoint_Small
Connections:
- net GND: no longer U1.3 (SD)
- net LM7705_SD: now reaches U4.23 (10_(D10))
- net LM7705_SD: now also U1.3 (SD), TP29.1
Other:
- moved on the sheet: D2, R3
Changed lines of the file:
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@@
 	)
 	(junction
+		(at 50.8 229.87)
+		(diameter 0)
+		(color 0 0 0 0)
+	)
+	(junction
 		(at 246.38 248.92)
 		(diameter 0)
@@
 	)
 	(junction
-		(at 52.07 229.87)
-		(diameter 0)
-		(color 0 0 0 0)
-	)
-	(junction
 		(at 349.25 100.33)
 		(diameter 0)
@@
 	(wire
 		(pts
-			(xy 52.07 229.87) (xy 44.45 229.87)
-		)
-		(stroke
-			(width 0)
-			(type default)
-		)
-	)
-	(wire
-		(pts
 			(xy 365.76 90.17) (xy 378.46 90.17)
 		)
@@
 	(wire
 		(pts
+			(xy 50.8 229.87) (xy 44.45 229.87)
+		)
+		(stroke
+			(width 0)
+			(type default)
+		)
+	)
+	(wire
+		(pts
 			(xy 148.59 177.8) (xy 151.13 177.8)
 		)
@@
 	(wire
 		(pts
-			(xy 38.1 130.81) (xy 25.4 130.81)
-		)
-		(stroke
-			(width 0)
-			(type default)
-		)
-	)
-	(wire
-		(pts
 			(xy 316.23 109.22) (xy 323.85 109.22)
 		)
@@
 	(wire
 		(pts
+			(xy 77.47 63.5) (xy 90.17 63.5)
+		)
+		(stroke
+			(width 0)
+			(type default)
+		)
+	)
+	(wire
+		(pts
 			(xy 186.69 240.03) (xy 208.28 240.03)
 		)
@@
 	(wire
 		(pts
-			(xy 77.47 63.5) (xy 93.98 63.5)
-		)
-		(stroke
-			(width 0)
-			(type default)
-		)
-	)
-	(wire
-		(pts
 			(xy 29.21 142.24) (xy 29.21 140.97)
 		)
@@
 	(wire
 		(pts
-			(xy 52.07 245.11) (xy 53.34 245.11)
+			(xy 50.8 245.11) (xy 53.34 245.11)
 		)
 		(stroke
@@
 	(wire
 		(pts
-			(xy 52.07 229.87) (xy 54.61 229.87)
-		)
-		(stroke
-			(width 0)
-			(type default)
-		)
-	)
-	(wire
-		(pts
 			(xy 140.97 256.54) (xy 140.97 257.81)
 		)
@@
 	(wire
 		(pts
+			(xy 25.4 130.81) (xy 38.1 130.81)
+		)
+		(stroke
+			(width 0)
+			(type default)
+		)
+	)
+	(wire
+		(pts
 			(xy 358.14 100.33) (xy 358.14 102.87)
 		)
@@
 	(wire
 		(pts
+			(xy 50.8 229.87) (xy 54.61 229.87)
+		)
+		(stroke
+			(width 0)
+			(type default)
+		)
+	)
+	(wire
+		(pts
 			(xy 151.13 170.18) (xy 149.86 170.18)
 		)
@@
 		)
 	)
+	(label "LM7705_SD"
+		(at 25.4 130.81 0)
+		(effects
+			(font
+				(size 1.27 1.27)
+			)
+			(justify left bottom)
+		)
+	)
 	(label "IN1"
 		(at 91.44 252.73 180)
@@
 		)
 	)
+	(label "LM7705_SD"
+		(at 90.17 63.5 180)
+		(effects
+			(font
+				(size 1.27 1.27)
+			)
+			(justify right bottom)
+		)
+	)
 	(label "CH5"
 		(at 316.23 82.55 0)
@@
 		(on_board yes)
 		(dnp no)
-		(fields_autoplaced yes)
 		(property "Reference" "U2"
 			(at 50.8 215.5824 0)
@@
 	(symbol
 		(lib_id "Connector:TestPoint_Small")
+		(at 90.17 63.5 0)
+		(unit 1)
+		(exclude_from_sim no)
+		(in_bom yes)
+		(on_board yes)
+		(dnp no)
+		(property "Reference" "TP29"
+			(at 91.186 63.5 0)
+			(effects
+				(font
+					(size 1.27 1.27)
+				)
+				(justify left)
+			)
+		)
+		(property "Value" "TestPoint_Small"
+			(at 91.44 64.7699 0)
+			(effects
+				(font
+					(size 1.27 1.27)
+				)
+				(justify left)
+				(hide yes)
+			)
+		)
+		(property "Footprint" "TestPoint:TestPoint_Keystone_5000-5004_Miniature"
+			(at 95.25 63.5 0)
+			(effects
+				(font
+					(size 1.27 1.27)
+				)
+				(hide yes)
+			)
+		)
+		(property "Datasheet" "~"
+			(at 95.25 63.5 0)
+			(effects
+				(font
+					(size 1.27 1.27)
+				)
+				(hide yes)
+			)
+		)
+		(property "Description" "test point"
+			(at 90.17 63.5 0)
+			(effects
+				(font
+					(size 1.27 1.27)
+				)
+				(hide yes)
+			)
+		)
+		(pin "1"
+		)
+		(instances
+			(project "phoenix-main-board"
+				(path "/8c64b4e9-9831-47d6-b522-c6dcea8b461a"
+					(reference "TP29")
+					(unit 1)
+				)
+			)
+		)
+	)
+	(symbol
+		(lib_id "Connector:TestPoint_Small")
 		(at 77.47 48.26 0)
 		(unit 1)
@@
 	(symbol
 		(lib_id "Device:R")
-		(at 52.07 233.68 180)
+		(at 50.8 233.68 180)
 		(unit 1)
 		(exclude_from_sim no)
@@
 		(dnp no)
 		(property "Reference" "R3"
-			(at 53.086 232.664 0)
+			(at 51.816 232.664 0)
 			(effects
 				(font
@@
 		)
 		(property "Value" "75"
-			(at 52.324 235.712 90)
+			(at 51.054 235.712 90)
 			(effects
 				(font
@@
 		)
 		(property "Footprint" "Resistor_SMD:R_0603_1608Metric"
-			(at 53.848 233.68 90)
+			(at 52.578 233.68 90)
 			(effects
 				(font
@@
 		)
 		(property "Datasheet" "~"
-			(at 52.07 233.68 0)
+			(at 50.8 233.68 0)
 			(effects
 				(font
@@
 		)
 		(property "Description" "Resistor"
-			(at 52.07 233.68 0)
+			(at 50.8 233.68 0)
 			(effects
 				(font
@@
 	(symbol
 		(lib_id "Device:LED")
-		(at 52.07 241.3 90)
+		(at 50.8 241.3 90)
 		(unit 1)
 		(exclude_from_sim no)
@@
 		(dnp no)
 		(property "Reference" "D2"
-			(at 52.578 238.506 90)
+			(at 51.308 238.506 90)
 			(effects
 				(font
@@
 		)
 		(property "Value" "GreenLED"
-			(at 50.292 237.49 0)
+			(at 49.022 237.49 0)
 			(effects
 				(font
@@
 		)
 		(property "Footprint" "LED_THT:LED_D5.0mm_Horizontal_O1.27mm_Z3.0mm"
-			(at 52.07 241.3 0)
+			(at 50.8 241.3 0)
 			(effects
 				(font
@@
 		)
 		(property "Datasheet" "~"
-			(at 52.07 241.3 0)
+			(at 50.8 241.3 0)
 			(effects
 				(font
@@
 		)
 		(property "Description" "Light emitting diode"
-			(at 52.07 241.3 0)
+			(at 50.8 241.3 0)
 			(effects
 				(font
@@
 		)
 		(property "Sim.Pins" "1=K 2=A"
-			(at 52.07 241.3 0)
+			(at 50.8 241.3 0)
 			(effects
 				(font
@@
 					(unit 1)
 				)
-			)
-		)
-	)
-	(symbol
-		(lib_id "power:GND")
-		(at 25.4 130.81 0)
-		(unit 1)
-		(exclude_from_sim no)
-		(in_bom yes)
-		(on_board yes)
-		(dnp no)
-		(property "Reference" "#PWR01"
-			(at 25.4 137.16 0)
-			(effects
-				(font
-					(size 1.27 1.27)
-				)
-				(hide yes)
-			)
-		)
-		(property "Value" "GND"
-			(at 25.4 134.874 0)
-			(effects
-				(font
-					(size 1.27 1.27)
-				)
-			)
-		)
-		(property "Footprint" ""
-			(at 25.4 130.81 0)
-			(effects
-				(font
-					(size 1.27 1.27)
-				)
-				(hide yes)
-			)
-		)
-		(property "Datasheet" ""
-			(at 25.4 130.81 0)
-			(effects
-				(font
-					(size 1.27 1.27)
-				)
-				(hide yes)
-			)
-		)
-		(property "Description" "Power symbol creates a global label with name \"GND\" , ground"
-			(at 25.4 130.81 0)
-			(effects
-				(font
-					(size 1.27 1.27)
-				)
-				(hide yes)
-			)
-		)
-		(pin "1"
-		)
-		(instances
-			(project "phoenix-main-board"
-				(path "/8c64b4e9-9831-47d6-b522-c6dcea8b461a"
-					(reference "#PWR01")
-					(unit 1)
-				)

Commit message: PCB: Complete V1.1.0-Tornado
Parts:
- removed JP1: SolderJumper_3_Bridged12, Jumper:SolderJumper-3_P1.3mm_Bridged2Bar12_Pad1.0x1.5mm, symbol Jumper:SolderJumper_3_Bridged12
- removed U3: TPS61222DCK, Package_TO_SOT_SMD:Texas_R-PDSO-G6, symbol Regulator_Switching:TPS61222DCK
- added C19, C20: 1uF, Capacitor_SMD:C_0603_1608Metric, symbol Device:C_Small
- added C21: 100nF, Capacitor_SMD:C_0603_1608Metric, symbol Device:C_Small
- added R21, R23, R24: 10k, Resistor_SMD:R_0603_1608Metric, symbol Device:R
- added R25: 1M, Resistor_SMD:R_0603_1608Metric, symbol Device:R
- added R26: 301k, Resistor_SMD:R_0603_1608Metric, symbol Device:R
- added TH3: GreenLEDThermistor, -ProjectLibrary:ThermistorWire, symbol Device:Thermistor
- added TH4: BlueLED Thermistor, -ProjectLibrary:ThermistorWire, symbol Device:Thermistor
- added TH5: GainStageThermistor, Resistor_SMD:R_0603_1608Metric, symbol Device:Thermistor
- added TP31, TP32, TP33, TP34: TestPoint_Small, TestPoint:TestPoint_Keystone_5000-5004_Miniature, symbol Connector:TestPoint_Small
- added U11: MCP41U83T, Package_DFN_QFN:Texas_RSA_VQFN-16-1EP_4x4mm_P0.65mm_EP2.7x2.7mm, symbol Potentiometer_Digital:MCP41U83x-xxxx-7N
- added U12: TPS7A2050, Package_TO_SOT_SMD:SOT-23-5, symbol -project-library:TPS7A2033
- added U3: MCP1640Bx-xCHY, Package_TO_SOT_SMD:SOT-23-6, symbol Regulator_Switching:MCP1640Bx-xCHY
- L1: footprint Inductor_SMD:L_0603_1608Metric -> Inductor_SMD:L_Wuerth_WE-TPC-3816
- R2: value 5 -> 0
- TH1: value EnclosureThermistor -> DriveStageThermistor
- TH2: footprint Connector_Wire:SolderWire-0.1sqmm_1x02_P3.6mm_D0.4mm_OD1mm_Relief -> -ProjectLibrary:ThermistorWire
- U6: value TPS7A2033DQN -> TPS7A2033
- renumbered PD2 to PD_Blue1, PD1 to PD_Green1
Connections:
- net +3.3V: no longer C1.1, C3.1, L1.1
- net +3.3VA: now also U11.16 (V_{DD})
- net +5V: now also U2.7, U2.8, C20.1, C21.1, TP31.1, U12.5 (OUT); no longer C8.1, TP12.1
- net EnablePower: now also U3.3 (EN)
- net GND: now also C19.2, C20.2, C21.2, R26.2, TH3.2, TH4.2, TH5.2, U11.1 (SDO/A1), U11.10 (V_{SS}), U11.17 (EP), U11.4 (~{CS}/A0), U11.6 (DGND), U12.2 (GND), U3.2 (GND)
- net SCL: now also U11.2 (SCK/SCL)
- net SDA: now also U11.3 (SDI/SDA)
- net Thermistor_On: now also R21.1, R23.1, R24.1
- net at L1.2: now also U3.1 (SW)
- net at U8.15 (W2): no longer RFB1.2
- net at U8.3 (W1): now also RFB1.2; no longer RFB2.2
- net PD_Green_SIG: now reaches U8.4 (B1)
- net PD_Green_SIG: now also R19.2, R4.1, U7.1 (OUT_A)
- net VBAT: now reaches TP13.1, U4.17 (VBAT)
- net VBAT: now also C1.1, C3.1, L1.1, U3.6 (V_{IN})
- net CH0: no longer names the net of TP24.1, U9.5 (CH0)
- net CH0: now also C18.1, R20.1; no longer R14.2, R15.1
- net CH1: no longer names the net of TP25.1, U9.6 (CH1)
- net CH1: now also C17.1, R19.1; no longer R17.2, TH1.1
- net CH2 renamed TH_GAIN
- net TH_GAIN: now also R24.2, TH5.1; no longer R18.2, TH2.1
- net CH3 renamed TH_DRV
- net TH_DRV: now also R17.2, TH1.1, TP32.1
- net CH4 renamed TH_BLU
- net TH_BLU: now also R23.2, TH4.1; no longer C18.1, R20.1
- net CH5 renamed TH_GRN
- net TH_GRN: now also R21.2, TH3.1; no longer C17.1, R19.1
- net CH6 renamed TH_SMP
- net TH_SMP: now also R18.2, TH2.1, TP33.1
- net CH7 renamed TH_REF
- net TH_REF: now also R14.2, R15.1, TP34.1
- removed net PD1_SIG: R20.2, R4.1, U7.1 (OUT_A), U8.16 (A2)
- net PD2_SIG renamed PD_Blue_SIG
- net PD_Blue_SIG: now also R20.2, U11.7 (P0B); no longer R19.2, U8.2 (A1)
- new net: R25.2, R26.1, U3.4 (V_{FB})
- new net: RFB2.2, U11.8 (P0W)
- new net 5.2V BOOST: C19.1, C8.1, R25.1, TP12.1, U12.1 (IN), U12.3 (EN), U3.5 (V_{OUT})
- no-connect marks 7 -> 10
Other:
- note added: "5V Boost"
- note added: "5V Ripple Rejection LDO"
- note added: "Inductor is Wuerth 744031004"
- note added: "Still have a number of these left so will use the 5242 for now Can go to 5241 in the future"
- note removed: "5V Charge Pump"
- moved on the sheet: C10, C11, C17, C18, C8, D1, D2, L1, R1, R14, R15, R17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
